Commit message: Update visical.xacro

File: visical_description/urdf/visical.xacro (robot description, xacro)
@@ -244,4 +244,10 @@
   </collision>
 </link>
+<link name="camera_link_optical"></link>
+<joint name="camera_optical_joint" type="fixed">
+  <origin xyz="-0.013 0 0.0075" rpy="0 ${-pi/2} 0"/>
+  <parent link="camera_1"/>
+  <child link="camera_link_optical"/>
+</joint>
 <link name="lidar_1">
   <inertial>
@@ -280,5 +286,5 @@
   <parent link="base_link"/>
   <child link="left_front_wheel_1"/>
-  <axis xyz="0.0 -1.0 0.0"/>
+  <axis xyz="0.0 1.0 0.0"/>
 </joint>
 <joint name="Rev4" type="continuous">
@@ -286,5 +292,5 @@
   <parent link="base_link"/>
   <child link="left_back_wheel_1"/>
-  <axis xyz="0.0 -1.0 0.0"/>
+  <axis xyz="0.0 1.0 0.0"/>
 </joint>
 <joint name="Rev5" type="continuous">
@@ -334,3 +340,8 @@
   <child link="lidar_1"/>
 </joint>
+<gazebo>
+ <plugin filename="libgazebo_ros_control.so" name="gazebo_ros_control">
+      <robotNamespace>/visical</robotNamespace>
+    </plugin>
+</gazebo>
 </robot>
