Commit message: Update materials.xacro

File: visical_description/urdf/materials.xacro (robot description, xacro)
@@ -4,3 +4,15 @@
   <color rgba="0.700 0.700 0.700 1.000"/>
 </material>
+<material name="Black">
+ <color rgba="0.0 0.0 0.0 1.0"/>
+</material>
+<material name="White">
+ <color rgba="1.0 1.0 1.0 1.0"/>
+</material>
+<material name="Blue">
+ <color rgba="0.0 0.0 1.0 1.0"/>
+</material>
+<material name="Green">
+ <color rgba="0.0 1.0 0.0 1.0"/>
+</material>
 </robot>
